File: hardware copy/motoko_ice_dragon.brd (EAGLE design)
At the start: 93 x 88 mm, 119 parts, among them IC2 LM2937, Q1 8MHz, Q10 20mA/30V, Q11 20mA/30V, Q2 BSS138TOP, Q3 BSS138TOP, Q4 20mA/30V, Q5 20mA/30V, Q6 20mA/30V, Q7 20mA/30V, Q8 20mA/30V, Q9 20mA/30V, U1 MP6540HA, U2 STM32_STM32F722XX, U3 MP6540HA

Commit message: main board
Parts:
- removed L_ENCODER1: (no value), con-lstb:MA04-1
- removed R37, R4, R40, R41: 4k7, resistor:M0805
- added R_ENCODER: (no value), con-lstb:MA04-1
Connections:
- net +3V3: now also R_ENCODER.4; no longer L_ENCODER1.4, R37.1, R4.1, R40.1, R41.1
- net GND: now also R_ENCODER.1; no longer L_ENCODER1.1
- net L_SCL: no longer R37.2
- net L_SDA: no longer R4.2
- net R_SCL: now also R_ENCODER.3; no longer L_ENCODER1.3, R41.2
- net R_SDA: now also R_ENCODER.2; no longer L_ENCODER1.2, R40.2
Routing:
- net +3V3: track 418.3 -> 405.0 mm, vias 10 -> 9
- net GND: track 604.3 -> 614.2 mm, vias 63 -> 60
- net L_SDA: track 26.1 -> 23.0 mm
- net L_SCL: track 22.7 -> 19.8 mm
- net R_SCL: track 20.8 -> 18.6 mm
- net R_SDA: track 23.7 -> 21.7 mm

Commit message: main board
Parts:
- removed C10, C12: 10uF, resistor:C0805
- removed C11, C9: 100n, resistor:C0805
- removed IC2: LM2937, linear:TO263-3
- removed R_ENCODER: (no value), con-lstb:MA04-1
- added C39, C41, C42: 100n, resistor:C0805
- added C40, C43, C44: 10uF, resistor:C0805
- added L1: 4.7uH, TYS50204R7N-10, SparkFun-Coils:CR54
- added L_ENCODER1: (no value), con-lstb:MA04-1
- added R37, R4, R40, R41: 4k7, resistor:M0805
- added U4: AP63203, SparkFun-IC-Power:SOT23-6
Connections:
- new net N$22: C39.2, U4.6
- new net N$26: C39.1, L1.P$1, U4.5
- net +3V3: now also C42.2, C43.2, C44.2, L1.P$2, L_ENCODER1.4, R37.1, R4.1, R40.1, R41.1, U4.1; no longer C11.1, C12.1, IC2.3, R_ENCODER.4
- net GND: now also C40.1, C41.1, C42.1, C43.1, C44.1, L_ENCODER1.1, U4.4; no longer C10.2, C11.2, C12.2, C9.2, IC2.2, R_ENCODER.1
- net L_SCL: now also R37.2
- net L_SDA: now also R4.2
- net R_SCL: now also L_ENCODER1.3, R41.2; no longer R_ENCODER.3
- net R_SDA: now also L_ENCODER1.2, R40.2; no longer R_ENCODER.2
- net VCC: now also C40.2, C41.2, U4.2, U4.3; no longer C10.1, C9.1, IC2.1
Routing:
- net GND: track 614.2 -> 584.3 mm
- net +3V3: track 405.0 -> 424.4 mm, vias 9 -> 10
- net N$26: track 0.00 -> 9.14 mm
- net VCC: track 181.0 -> 177.5 mm, vias 11 -> 12
- net L_SDA: track 23.0 -> 26.1 mm
- net L_SCL: track 19.8 -> 22.7 mm
- net N$22: track 0.00 -> 2.61 mm
- net R_SCL: track 18.6 -> 20.8 mm
- net R_SDA: track 21.7 -> 23.7 mm
