File: hardware/motoko_ice_dragon.brd (EAGLE design)
At the start: 93 x 88 mm, 119 parts, among them IC2 LM2937, Q1 8MHz, Q10 20mA/30V, Q11 20mA/30V, Q2 BSS138TOP, Q3 BSS138TOP, Q4 20mA/30V, Q5 20mA/30V, Q6 20mA/30V, Q7 20mA/30V, Q8 20mA/30V, Q9 20mA/30V, U1 MP6540HA, U2 STM32_STM32F722XX, U3 MP6540HA

Commit message: main board
Parts:
- removed C10, C12: 10uF, resistor:C0805
- removed C11, C9: 100n, resistor:C0805
- removed IC2: LM2937, linear:TO263-3
- added C39, C41, C42: 100n, resistor:C0805
- added C40, C43, C44: 10uF, resistor:C0805
- added L1: 4.7uH, TYS50204R7N-10, SparkFun-Coils:CR54
- added U4: AP63203, SparkFun-IC-Power:SOT23-6
Connections:
- new net N$22: C39.2, U4.6
- new net N$26: C39.1, L1.P$1, U4.5
- net +3V3: now also C42.2, C43.2, C44.2, L1.P$2, U4.1; no longer C11.1, C12.1, IC2.3
- net GND: now also C40.1, C41.1, C42.1, C43.1, C44.1, U4.4; no longer C10.2, C11.2, C12.2, C9.2, IC2.2
- net VCC: now also C40.2, C41.2, U4.2, U4.3; no longer C10.1, C9.1, IC2.1
Routing:
- net GND: track 604.3 -> 584.3 mm, vias 63 -> 60
- net N$26: track 0.00 -> 9.14 mm
- net +3V3: track 418.3 -> 424.4 mm
- net VCC: track 181.0 -> 177.5 mm, vias 11 -> 12
- net N$22: track 0.00 -> 2.61 mm

Commit message: identification, sensors calibrations
Connections:
- net L_SCL: now also L_ENCODER.2, R4.2, U2.62; no longer L_ENCODER.3, R37.2, U2.61
- net L_SDA: now also L_ENCODER.3, R37.2, U2.61; no longer L_ENCODER.2, R4.2, U2.62
Routing:
- net L_SDA: track 26.1 -> 22.7 mm
- net L_SCL: track 22.7 -> 26.1 mm
