File: hardware/motoko_ice_dragon.brd (EAGLE design)
At the start: 93 x 88 mm, 122 parts, among them Q1 8MHz, Q10 20mA/30V, Q11 20mA/30V, Q2 BSS138TOP, Q3 BSS138TOP, Q4 20mA/30V, Q5 20mA/30V, Q6 20mA/30V, Q7 20mA/30V, Q8 20mA/30V, Q9 20mA/30V, U1 MP6540HA, U2 STM32_STM32F722XX, U3 MP6540HA, U4 AP63203

Commit message: board rev 2
Parts:
- removed C14: 10n, resistor:C0805
- removed LSM6DS1: ST_L3GD20H, motoko_5_0:ST_LGA16L
- added C9: 100n, resistor:C0805
- added FD1, FD2, FD3, FD4, FD5, FD6, FD7, FD8, FD9: FIDUCIAL1X2, SparkFun-Aesthetics:FIDUCIAL-1X2
- added JP2: boot, jumper:JP1
- added LED10: (no value), led:CHIPLED_1206
- added R38: 330, resistor:M0805
- added R39: 4k7, resistor:M0805
- added R42, R43: 4k7, rcl:M0805
- added U$3: LSM6DSM, my_library:LGA14L
- added U$4: 24LC24_SOT23, my_library:SOT23
- R1, R36: device resistor:M0805 -> rcl:M1206
- moved LED9 70.0 mm to (17.0, 15.0), turned to 270 degrees
- moved R9 61.0 mm to (22.0, 15.0), flipped to the bottom
- moved LED8 37.0 mm to (86.0, 46.0)
- moved R25 36.9 mm to (81.5, 46.1)
- moved C26 7.42 mm to (13.7, 44.9), turned to 270 degrees
- moved LED1 3.00 mm to (86.0, 10.0)
- moved LED2 3.00 mm to (86.0, 20.0)
- moved LED3 3.00 mm to (86.0, 30.0)
- moved LED4 3.00 mm to (86.0, 40.0)
- moved LED5 3.00 mm to (86.0, 56.0)
- moved LED6 3.00 mm to (86.0, 66.0)
- moved LED7 3.00 mm to (86.0, 76.0)
- moved R18 0.91 mm to (81.2, 49.0)
- moved L1 0.30 mm to (14.0, 44.5)
Connections:
- removed net N$6: C14.2, LSM6DS1.P$14
- new net LED_2: R9.2, U2.1
- new net LED_3: R38.2, U2.60
- new net MEM_SCL: R42.2, U$4.P$1, U2.85
- new net MEM_SDA: R43.2, U$4.P$3, U2.84
- new net N$11: LED10.A, R38.1
- net +3V3: now also C9.1, JP2.2, R42.1, R43.1, U$3.P$12, U$3.P$5, U$3.P$8, U$4.P$4; no longer LSM6DS1.P$1, LSM6DS1.P$16, LSM6DS1.P$5, R9.2
- net BOOT: now also JP2.1, R39.2
- net GND: now also C9.2, LED10.C, LED9.C, R39.1, U$3.P$1, U$3.P$2, U$3.P$3, U$3.P$6, U$3.P$7, U$4.P$2, U$4.P$5; no longer C14.1, LSM6DS1.P$10, LSM6DS1.P$11, LSM6DS1.P$12, LSM6DS1.P$13, LSM6DS1.P$15, LSM6DS1.P$4, LSM6DS1.P$8, LSM6DS1.P$9
- net KEY: now also U2.3; no longer U2.2
- net LED_1: now also U2.2; no longer U2.1
- net LINE_LED: no longer LED9.C
- net SCL: now also U$3.P$13; no longer LSM6DS1.P$2
- net SDA: now also U$3.P$14; no longer LSM6DS1.P$3
Routing:
- net LED_2: track 0.00 -> 37.2 mm, vias 0 -> 3
- net BOOT: track 0.00 -> 30.4 mm, vias 0 -> 3
- net LED_3: track 0.00 -> 28.9 mm, vias 0 -> 3
- net LINE_LED: track 110.9 -> 95.6 mm
- net +3V3: track 424.4 -> 436.8 mm, vias 10 -> 11
- net MEM_SCL: track 0.00 -> 7.46 mm, vias 0 -> 1
- net GND: track 584.3 -> 591.3 mm, vias 60 -> 61
- net MEM_SDA: track 0.00 -> 5.37 mm, vias 0 -> 1
- net N$6: track 5.03 -> 0.00 mm
- net SDA: track 16.8 -> 20.2 mm
- net SCL: track 17.9 -> 20.8 mm
- net N$14: track 1.79 -> 4.42 mm
- net N$17: track 2.05 -> 4.53 mm
- net N$15: track 1.74 -> 4.22 mm
- net N$19: track 1.97 -> 4.33 mm
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
Commit message: gyro tests
Connections:
- net L_SCL: now also L_ENCODER.3, R37.2, U2.61; no longer L_ENCODER.2, R4.2, U2.62
- net L_SDA: now also L_ENCODER.2, R4.2, U2.62; no longer L_ENCODER.3, R37.2, U2.61
Routing:
- net L_SDA: track 22.7 -> 26.1 mm
- net L_SCL: track 26.1 -> 22.7 mm
Changed lines of the file:
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@@
 <wire x1="9.144" y1="47.8892" x2="9.718" y2="48.4632" width="0.6096" layer="16"/>
 </signal>
-<signal name="L_SDA">
-<contactref element="U2" pad="61"/>
+<signal name="L_SCL">
 <contactref element="L_ENCODER" pad="3"/>
-<wire x1="31.51065625" y1="53.456259375" x2="31.51065625" y2="63.83265625" width="0.3048" layer="1"/>
+<wire x1="31.51065625" y1="54.2544" x2="31.51065625" y2="63.83265625" width="0.3048" layer="1"/>
 <wire x1="31.51065625" y1="63.83265625" x2="33.6992" y2="66.0212" width="0.3048" layer="1"/>
 <contactref element="R37" pad="2"/>
 <wire x1="33.6992" y1="66.0212" x2="36.6736" y2="66.0212" width="0.3048" layer="1"/>
 <wire x1="36.6736" y1="66.0212" x2="36.6876" y2="66.0072" width="0.3048" layer="1"/>
+<contactref element="U2" pad="61"/>
 <wire x1="35.9246625" y1="49.042253125" x2="31.51065625" y2="53.456259375" width="0.3048" layer="1"/>
-</signal>
-<signal name="L_SCL">
-<contactref element="U2" pad="62"/>
-<wire x1="35.5834125" y1="48.701003125" x2="30.956" y2="53.328415625" width="0.3048" layer="1"/>
-<wire x1="30.956" y1="53.328415625" x2="30.956" y2="66.008" width="0.3048" layer="1"/>
-<wire x1="33.5092" y1="68.5612" x2="30.956" y2="66.008" width="0.3048" layer="1"/>
-<contactref element="L_ENCODER" pad="2"/>
-<contactref element="R4" pad="2"/>
-<wire x1="33.6992" y1="68.5612" x2="33.7892" y2="68.6512" width="0.3048" layer="1"/>
-<wire x1="33.7892" y1="68.6512" x2="36.6876" y2="68.6512" width="0.3048" layer="1"/>
-<wire x1="33.6992" y1="68.5612" x2="33.5092" y2="68.5612" width="0.3048" layer="1"/>
+<wire x1="31.51065625" y1="53.456259375" x2="31.51065625" y2="54.2544" width="0.3048" layer="1"/>
 </signal>
 <signal name="N$9">
@@
 <wire x1="31.25" y1="37.6348" x2="31.25" y2="36.9" width="0.3048" layer="1"/>
 </signal>
+<signal name="L_SDA">
+<contactref element="L_ENCODER" pad="2"/>
+<contactref element="R4" pad="2"/>
+<wire x1="30.956" y1="54.2544" x2="30.956" y2="66.008" width="0.3048" layer="1"/>
+<wire x1="33.5092" y1="68.5612" x2="30.956" y2="66.008" width="0.3048" layer="1"/>
+<wire x1="33.6992" y1="68.5612" x2="33.7892" y2="68.6512" width="0.3048" layer="1"/>
+<wire x1="33.7892" y1="68.6512" x2="36.6876" y2="68.6512" width="0.3048" layer="1"/>
+<wire x1="33.6992" y1="68.5612" x2="33.5092" y2="68.5612" width="0.3048" layer="1"/>
+<contactref element="U2" pad="62"/>
+<wire x1="35.5834125" y1="48.701003125" x2="30.956" y2="53.328415625" width="0.3048" layer="1"/>
+<wire x1="30.956" y1="53.328415625" x2="30.956" y2="54.2544" width="0.3048" layer="1"/>
+</signal>
 </signals>
