File: hardware/v0/motoko_ice_dragon.brd (EAGLE design)
At the start: 93 x 88 mm, 138 parts, among them Q1 8MHz, Q10 20mA/30V, Q11 20mA/30V, Q2 BSS138TOP, Q3 BSS138TOP, Q4 20mA/30V, Q5 20mA/30V, Q6 20mA/30V, Q7 20mA/30V, Q8 20mA/30V, Q9 20mA/30V, U1 MP6540HA, U2 STM32_STM32F722XX, U3 MP6540HA, U4 AP63203

Commit message: boards
Parts:
- added D1: 3A/40V/500mV, SparkFun-DiscreteSemi:SMA-DIODE
- added L_ENCODER2: (no value), con-lstb:MA04-1
- added R44: 1k5, resistor:M0805
- moved FD2 9.17 mm to (82.6, 51.5)
- moved FD1 8.50 mm to (83.9, 51.2)
- moved LED1 1.00 mm to (86.0, 11.0)
- moved LED2 1.00 mm to (86.0, 21.0)
- moved LED3 1.00 mm to (86.0, 31.0)
- moved LED4 1.00 mm to (86.0, 41.0)
- moved LED5 1.00 mm to (86.0, 55.0)
- moved LED6 1.00 mm to (86.0, 65.0)
- moved LED7 1.00 mm to (86.0, 75.0)
- moved LED8 1.00 mm to (86.0, 45.0)
Connections:
- new net N$28: D1.A, L_ENCODER2.4
- new net USBDM: L_ENCODER2.3, U2.70
- new net USBDP: L_ENCODER2.2, R44.1, U2.71
- net +3V3: now also R44.2
- net GND: now also L_ENCODER2.1
- net VCC: now also D1.C
Routing:
- net USBDP: track 0.00 -> 63.2 mm, vias 0 -> 2
- net USBDM: track 0.00 -> 61.9 mm, vias 0 -> 2
- net +3V3: track 436.8 -> 443.7 mm
- net GND: track 591.3 -> 596.2 mm
- net VCC: track 177.5 -> 174.9 mm
- net N$28: track 0.00 -> 2.57 mm
- net LINE_LED: track 95.6 -> 93.8 mm
- net N$15: track 4.22 -> 3.22 mm
- net N$20: track 4.18 -> 3.18 mm
- net N$19: track 4.33 -> 3.33 mm
- net N$18: track 4.53 -> 3.53 mm
- net N$16: track 4.14 -> 3.14 mm
- net N$14: track 4.42 -> 3.42 mm
