File: hardware/v0/motoko_ice_dragon.sch (EAGLE design)
At the start: 138 parts, among them Q1 8MHz, Q10 20mA/30V, Q11 20mA/30V, Q2 BSS138TOP, Q3 BSS138TOP, Q4 20mA/30V, Q5 20mA/30V, Q6 20mA/30V, Q7 20mA/30V, Q8 20mA/30V, Q9 20mA/30V, U1 MP6540HA, U2 STM32_STM32F722XX, U3 MP6540HA, U4 AP63203

Commit message: boards
Parts:
- added D1: 3A/40V/500mV, SparkFun-DiscreteSemi:DIODE-SCHOTTKY-B340A
- added L_ENCODER2: (no value), con-lstb:MA04-1
- added R44: 1k5, resistor:R-EU_M0805
Connections:
- new net N$28: D1.A, L_ENCODER2.4
- new net USBDM: L_ENCODER2.3, U2B.PA_11
- new net USBDP: L_ENCODER2.2, R44.1, U2B.PA12
- net +3V3: now also R44.2
- net GND: now also L_ENCODER2.1
- net VCC: now also D1.C
Changed lines of the file:
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@@
 <?xml version="1.0" encoding="utf-8"?>
 <!DOCTYPE eagle SYSTEM "eagle.dtd">
-<eagle version="9.6.2">
+<eagle version="9.6.0">
 <drawing>
 <settings>
@@
 <setting verticaltext="up"/>
 </settings>
-<grid distance="0.1" unitdist="inch" unit="inch" style="lines" multiple="1" display="no" altdistance="0.01" altunitdist="inch" altunit="inch"/>
+<grid distance="0.05" unitdist="inch" unit="inch" style="lines" multiple="1" display="no" altdistance="0.01" altunitdist="inch" altunit="inch"/>
 <layers>
 <layer number="1" name="Top" color="4" fill="1" visible="no" active="no"/>
@@
 <part name="GND56" library="supply1" library_urn="urn:adsk.eagle:library:371" deviceset="GND" device=""/>
 <part name="+3V59" library="supply1" library_urn="urn:adsk.eagle:library:371" deviceset="+3V3" device=""/>
+<part name="L_ENCODER2" library="con-lstb" library_urn="urn:adsk.eagle:library:162" deviceset="MA04-1" device="" package3d_urn="urn:adsk.eagle:package:8337/1"/>
+<part name="P+9" library="supply1" library_urn="urn:adsk.eagle:library:371" deviceset="VCC" device=""/>
+<part name="GND57" library="supply1" library_urn="urn:adsk.eagle:library:371" deviceset="GND" device=""/>
+<part name="D1" library="SparkFun-DiscreteSemi" deviceset="DIODE-SCHOTTKY" device="-B340A" value="3A/40V/500mV"/>
+<part name="R44" library="resistor" library_urn="urn:adsk.eagle:library:348" deviceset="R-EU_" device="M0805" package3d_urn="urn:adsk.eagle:package:26079/1" value="1k5"/>
+<part name="+3V60" library="supply1" library_urn="urn:adsk.eagle:library:371" deviceset="+3V3" device=""/>
 </parts>
 <sheets>
@@
 <attribute name="NAME" x="259.08" y="154.94" size="1.778" layer="95" font="vector" rot="R90"/>
 </instance>
-<instance part="FD1" gate="G$1" x="340.36" y="124.46" smashed="yes"/>
-<instance part="FD2" gate="G$1" x="340.36" y="119.38" smashed="yes"/>
-<instance part="FD3" gate="G$1" x="340.36" y="114.3" smashed="yes"/>
-<instance part="FD4" gate="G$1" x="340.36" y="109.22" smashed="yes"/>
-<instance part="FD5" gate="G$1" x="340.36" y="104.14" smashed="yes"/>
+<instance part="FD1" gate="G$1" x="355.6" y="124.46" smashed="yes"/>
+<instance part="FD2" gate="G$1" x="355.6" y="119.38" smashed="yes"/>
+<instance part="FD3" gate="G$1" x="355.6" y="114.3" smashed="yes"/>
+<instance part="FD4" gate="G$1" x="355.6" y="109.22" smashed="yes"/>
+<instance part="FD5" gate="G$1" x="355.6" y="104.14" smashed="yes"/>
 <instance part="LED9" gate="G$1" x="262.89" y="62.23" smashed="yes">
 <attribute name="NAME" x="266.446" y="57.658" size="1.778" layer="95" rot="R90"/>
@@
 <attribute name="VALUE" x="281.94" y="46.99" size="1.778" layer="96"/>
 </instance>
-<instance part="FD6" gate="G$1" x="349.25" y="124.46" smashed="yes"/>
-<instance part="FD7" gate="G$1" x="349.25" y="119.38" smashed="yes"/>
-<instance part="FD8" gate="G$1" x="349.25" y="114.3" smashed="yes"/>
+<instance part="FD6" gate="G$1" x="364.49" y="124.46" smashed="yes"/>
+<instance part="FD7" gate="G$1" x="364.49" y="119.38" smashed="yes"/>
+<instance part="FD8" gate="G$1" x="364.49" y="114.3" smashed="yes"/>
 <instance part="U$3" gate="G$1" x="57.15" y="97.79" smashed="yes"/>
 <instance part="GND26" gate="1" x="64.77" y="74.93" smashed="yes">
@@
 <attribute name="VALUE" x="67.31" y="116.84" size="1.778" layer="96" rot="R90"/>
 </instance>
-<instance part="FD9" gate="G$1" x="349.25" y="109.22" smashed="yes"/>
+<instance part="FD9" gate="G$1" x="364.49" y="109.22" smashed="yes"/>
 <instance part="U$4" gate="G$1" x="238.76" y="114.3" smashed="yes"/>
 <instance part="+3V39" gate="G$1" x="223.52" y="127" smashed="yes">
@@
 <attribute name="VALUE" x="288.29" y="121.92" size="1.778" layer="96" rot="R90"/>
 </instance>
+<instance part="L_ENCODER2" gate="1" x="302.26" y="113.03" smashed="yes">
+<attribute name="VALUE" x="300.99" y="102.87" size="1.778" layer="96"/>
+</instance>
+<instance part="P+9" gate="VCC" x="323.85" y="128.27" smashed="yes">
+<attribute name="VALUE" x="321.31" y="125.73" size="1.778" layer="96" rot="R90"/>
+</instance>
+<instance part="GND57" gate="1" x="311.15" y="104.14" smashed="yes">
+<attribute name="VALUE" x="308.61" y="101.6" size="1.778" layer="96"/>
+</instance>
+<instance part="D1" gate="G$1" x="323.85" y="120.65" smashed="yes" rot="R90">
+<attribute name="NAME" x="321.818" y="118.11" size="1.778" layer="95" font="vector" rot="R90"/>
+</instance>
+<instance part="R44" gate="G$1" x="331.47" y="119.38" smashed="yes" rot="MR90">
+<attribute name="NAME" x="332.9686" y="115.57" size="1.778" layer="95" rot="MR90"/>
+<attribute name="VALUE" x="328.168" y="115.57" size="1.778" layer="96" rot="MR90"/>
+</instance>
+<instance part="+3V60" gate="G$1" x="331.47" y="128.27" smashed="yes">
+<attribute name="VALUE" x="328.93" y="123.19" size="1.778" layer="96" rot="R90"/>
+</instance>
 </instances>
 <busses>
@@
 <wire x1="290.83" y1="101.6" x2="290.83" y2="104.14" width="0.1524" layer="91"/>
 </segment>
+<segment>
+<pinref part="L_ENCODER2" gate="1" pin="1"/>
+<pinref part="GND57" gate="1" pin="GND"/>
+<wire x1="309.88" y1="107.95" x2="311.15" y2="107.95" width="0.1524" layer="91"/>
+<wire x1="311.15" y1="107.95" x2="311.15" y2="106.68" width="0.1524" layer="91"/>
+</segment>
 </net>
 <net name="VCC" class="0">
@@
 <wire x1="198.12" y1="163.83" x2="198.12" y2="156.21" width="0.1524" layer="91"/>
 </segment>
+<segment>
+<pinref part="D1" gate="G$1" pin="C"/>
+<pinref part="P+9" gate="VCC" pin="VCC"/>
+<wire x1="323.85" y1="123.19" x2="323.85" y2="125.73" width="0.1524" layer="91"/>
+</segment>
 </net>
 <net name="+3V3" class="0">
@@
 <wire x1="290.83" y1="111.76" x2="290.83" y2="124.46" width="0.1524" layer="91"/>
 </segment>
+<segment>
+<pinref part="R44" gate="G$1" pin="2"/>
+<pinref part="+3V60" gate="G$1" pin="+3V3"/>
+<wire x1="331.47" y1="124.46" x2="331.47" y2="125.73" width="0.1524" layer="91"/>
+</segment>
 </net>
 <net name="SCL" class="0">
@@
 </segment>
 </net>
+<net name="USBDP" class="0">
+<segment>
+<pinref part="L_ENCODER2" gate="1" pin="2"/>
+<label x="334.01" y="110.49" size="1.778" layer="95"/>
+<pinref part="R44" gate="G$1" pin="1"/>
+<wire x1="331.47" y1="114.3" x2="331.47" y2="110.49" width="0.1524" layer="91"/>
+<wire x1="331.47" y1="110.49" x2="309.88" y2="110.49" width="0.1524" layer="91"/>
+</segment>
+<segment>
+<pinref part="U2" gate="B" pin="PA12"/>
+<wire x1="110.49" y1="198.12" x2="105.41" y2="198.12" width="0.1524" layer="91"/>
+<label x="104.14" y="198.12" size="1.778" layer="95" rot="R180"/>
+</segment>
+</net>
+<net name="USBDM" class="0">
+<segment>
+<pinref part="L_ENCODER2" gate="1" pin="3"/>
+<wire x1="309.88" y1="113.03" x2="314.96" y2="113.03" width="0.1524" layer="91"/>
+<label x="316.23" y="113.03" size="1.778" layer="95"/>
+</segment>
+<segment>
+<pinref part="U2" gate="B" pin="PA_11"/>
+<wire x1="110.49" y1="200.66" x2="105.41" y2="200.66" width="0.1524" layer="91"/>
+<label x="104.14" y="200.66" size="1.778" layer="95" rot="R180"/>
+</segment>
+</net>
+<net name="N$28" class="0">
+<segment>
+<pinref part="L_ENCODER2" gate="1" pin="4"/>
+<wire x1="309.88" y1="115.57" x2="323.85" y2="115.57" width="0.1524" layer="91"/>
+<pinref part="D1" gate="G$1" pin="A"/>
+<wire x1="323.85" y1="118.11" x2="323.85" y2="115.57" width="0.1524" layer="91"/>
+</segment>
+</net>
