File: hardware/v1/motoko_ice_dragon_v1.brd (EAGLE design)
At the start: 100 x 80 mm, 121 parts, among them Q1 8MHz, Q10 20mA/30V, Q11 20mA/30V, Q2 BSS138TOP, Q4 20mA/30V, Q5 20mA/30V, Q6 20mA/30V, Q7 20mA/30V, Q8 20mA/30V, Q9 20mA/30V, U1 MP6540HA, U2 STM32_STM32F722XX, U3 MP6540HA, U4 AP63203, X1 FH12-12S-0.5SH, X2 FH12-12S-0.5SH, X3 52745-0490, X4 52745-0490, X5 52745-0490

Commit message: boards
Other:
- outline, holes or cut-outs redrawn
Changed lines of the file:
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@@
 <setting verticaltext="up"/>
 </settings>
-<grid distance="12" unitdist="mil" unit="mil" style="lines" multiple="1" display="yes" altdistance="5" altunitdist="mil" altunit="mil"/>
+<grid distance="1" unitdist="mm" unit="mm" style="lines" multiple="1" display="yes" altdistance="5" altunitdist="mil" altunit="mil"/>
 <layers>
 <layer number="1" name="Top" color="4" fill="1" visible="yes" active="yes"/>
@@
 <wire x1="81" y1="40" x2="60" y2="61" width="0" layer="20"/>
 <wire x1="60" y1="61" x2="60" y2="68" width="0" layer="20"/>
-<wire x1="60" y1="68" x2="85" y2="68" width="0" layer="20"/>
-<wire x1="85" y1="68" x2="87" y2="69" width="0" layer="20"/>
-<wire x1="87" y1="69" x2="87" y2="78" width="0" layer="20"/>
-<wire x1="87" y1="78" x2="85" y2="80" width="0" layer="20"/>
-<wire x1="85" y1="80" x2="15" y2="80" width="0" layer="20"/>
-<wire x1="15" y1="80" x2="13" y2="78" width="0" layer="20"/>
-<wire x1="13" y1="78" x2="13" y2="69" width="0" layer="20"/>
-<wire x1="13" y1="69" x2="15" y2="68" width="0" layer="20"/>
-<wire x1="15" y1="68" x2="40" y2="68" width="0" layer="20"/>
+<wire x1="60" y1="68" x2="87" y2="68" width="0" layer="20"/>
+<wire x1="87" y1="68" x2="90" y2="69" width="0" layer="20"/>
+<wire x1="90" y1="69" x2="90" y2="78" width="0" layer="20"/>
+<wire x1="90" y1="78" x2="87" y2="80" width="0" layer="20"/>
+<wire x1="87" y1="80" x2="13" y2="80" width="0" layer="20"/>
+<wire x1="13" y1="80" x2="10" y2="78" width="0" layer="20"/>
+<wire x1="10" y1="78" x2="10" y2="69" width="0" layer="20"/>
+<wire x1="10" y1="69" x2="13" y2="68" width="0" layer="20"/>
+<wire x1="13" y1="68" x2="40" y2="68" width="0" layer="20"/>
 <wire x1="40" y1="68" x2="40" y2="61" width="0" layer="20"/>
 <wire x1="40" y1="61" x2="18" y2="40" width="0" layer="20"/>
@@
 <wire x1="50" y1="1" x2="50" y2="86" width="0.2" layer="51"/>
 <wire x1="116" y1="15" x2="-19" y2="15" width="0.2" layer="51"/>
-<dimension x1="50" y1="86" x2="13" y2="86" x3="31.5" y3="64" textsize="1.778" layer="51"/>
-<dimension x1="50" y1="86" x2="87" y2="86" x3="68.5" y3="64" textsize="1.778" layer="51"/>
 <dimension x1="0" y1="0" x2="100" y2="0" x3="50" y3="-6.096" textsize="1.778" layer="51"/>
 <dimension x1="0" y1="0" x2="24.6888" y2="79.8576" x3="120.0912" y3="39.9288" textsize="1.778" layer="51" dtype="vertical"/>

Commit message: new foc
Parts:
- added U$5: DUCTED_FAN_35MM, my_library:DUCTED_FAN_35MM
- U$1, U$2: value BRUSHLESS_GIMBAL_MOTOR_WHEEL -> BRUSHLESS_MOTOR_WHEEL; device my_library:BRUSHLESS_GIMBAL_MOTOR_WHEEL -> my_library:BRUSHLESS_MOTOR_WHEEL
- moved U$2 14.9 mm to (86.0, 20.0), flipped to the bottom, turned to 0 degrees
- moved U$1 13.9 mm to (13.1, 19.7)
Routing:
- net R_YA: track 15.7 -> 27.4 mm
- net L_YC: track 15.2 -> 4.01 mm
- net R_YB: track 15.1 -> 26.3 mm
- net L_YB: track 14.8 -> 4.01 mm
- net R_YC: track 15.6 -> 25.5 mm
- net L_YA: track 14.4 -> 7.37 mm
- removed copper zone on layer 1, net GND
- removed copper zone on layer 16, net GND
