File: hardware/v1/motoko_ice_dragon_v1.sch (EAGLE design)
At the start: 121 parts, among them Q1 8MHz, Q10 20mA/30V, Q11 20mA/30V, Q2 BSS138TOP, Q4 20mA/30V, Q5 20mA/30V, Q6 20mA/30V, Q7 20mA/30V, Q8 20mA/30V, Q9 20mA/30V, U1 MP6540HA, U2 STM32_STM32F722XX, U3 MP6540HA, U4 AP63203, X1 FH12-12S-0.5SH, X2 FH12-12S-0.5SH, X3 52745-0490, X4 52745-0490, X5 52745-0490

Commit message: new foc
Parts:
- added U$5: DUCTED_FAN_35MM, my_library:DUCTED_FAN_35MM
- U$1, U$2: value BRUSHLESS_GIMBAL_MOTOR_WHEEL -> BRUSHLESS_MOTOR_WHEEL; device my_library:BRUSHLESS_GIMBAL_MOTOR_WHEEL -> my_library:BRUSHLESS_MOTOR_WHEEL
Changed lines of the file:
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@@
 <setting verticaltext="up"/>
 </settings>
-<grid distance="0.05" unitdist="inch" unit="inch" style="lines" multiple="1" display="no" altdistance="0.01" altunitdist="inch" altunit="inch"/>
+<grid distance="0.1" unitdist="inch" unit="inch" style="lines" multiple="1" display="no" altdistance="0.01" altunitdist="inch" altunit="inch"/>
 <layers>
 <layer number="1" name="Top" color="4" fill="1" visible="no" active="no"/>
@@
 <part name="LED7" library="led" library_urn="urn:adsk.eagle:library:259" deviceset="LED" device="CHIPLED_1206" package3d_urn="urn:adsk.eagle:package:15823/2"/>
 <part name="LED8" library="led" library_urn="urn:adsk.eagle:library:259" deviceset="LED" device="CHIPLED_1206" package3d_urn="urn:adsk.eagle:package:15823/2"/>
-<part name="U$1" library="my_library" deviceset="BRUSHLESS_GIMBAL_MOTOR_WHEEL" device=""/>
-<part name="U$2" library="my_library" deviceset="BRUSHLESS_GIMBAL_MOTOR_WHEEL" device=""/>
+<part name="U$1" library="my_library" deviceset="BRUSHLESS_MOTOR_WHEEL" device=""/>
+<part name="U$2" library="my_library" deviceset="BRUSHLESS_MOTOR_WHEEL" device=""/>
 <part name="C27" library="resistor" library_urn="urn:adsk.eagle:library:348" deviceset="C-EU" device="C0805" package3d_urn="urn:adsk.eagle:package:26137/1" value="100n"/>
 <part name="C35" library="resistor" library_urn="urn:adsk.eagle:library:348" deviceset="C-EU" device="C0805" package3d_urn="urn:adsk.eagle:package:26137/1" value="10uF"/>
@@
 <part name="+3V38" library="supply1" library_urn="urn:adsk.eagle:library:371" deviceset="+3V3" device=""/>
 <part name="GND28" library="supply1" library_urn="urn:adsk.eagle:library:371" deviceset="GND" device=""/>
+<part name="U$5" library="my_library" deviceset="DUCTED_FAN_35MM" device=""/>
 </parts>
 <sheets>
@@
 <attribute name="VALUE" x="242.57" y="68.58" size="1.778" layer="96"/>
 </instance>
+<instance part="U$5" gate="G$1" x="243.84" y="200.66" smashed="yes"/>
 </instances>
 <busses>
